File: pcb/fih.kicad_pcb (KiCad board)
At the start: 2 copper layers, 114.6 x 76.5 mm, 19 parts

Commit message: choc v2
Parts:
- S13: moved to F.Cu
- moved XX1 10.6 mm to (199.5, 133.0), turned to 90 degrees
- moved PWR1 7.07 mm to (193.5, 140.0)
- turned S13 to 180 degrees
Connections:
- net P2 renamed P21
- MCU1 pad 101: P1 -> RAW
- MCU1 pad 102: P0 -> GND
- MCU1 pad 103: GND -> RST
- MCU1 pad 104: GND -> VCC
- MCU1 pad 121: VCC -> GND
- MCU1 pad 122: RST -> GND
- MCU1 pad 123: GND -> P0
- MCU1 pad 124: RAW -> P1
Routing:
- net RST: track 34.8 -> 24.6 mm, vias 1 -> 0
- net RAW: track 51.3 -> 54.6 mm
- net matrix_index_bottom: track 64.8 -> 63.2 mm
- net matrix_index_home: track 77.0 -> 75.3 mm
- net matrix_index_top: track 89.7 -> 88.1 mm
- net matrix_middle_bottom: track 101.6 -> 100.0 mm
- net matrix_middle_top: track 127.1 -> 125.5 mm
- net matrix_inner_top: track 55.7 -> 54.1 mm
- net matrix_inner_home: track 42.7 -> 41.1 mm
- net matrix_middle_home: track 114.3 -> 112.7 mm
- net GND: track 42.9 -> 41.5 mm
